Commit message: feat: 简单机械臂完整建模

File: src/demo_urdf_pkg/urdf/simple_arm.urdf (robot description, URDF)
Before this commit: robot simple_arm, 1 links, 0 joints
Links:
- added link gripper_base_link, mass 1; collision box size=0.1 0.2 0.05; visual box size=0.1 0.2 0.05
- added link hand_left_link, mass 1; collision box size=0.1 0.2 0.05; visual box size=0.1 0.05 0.1
- added link hand_right_link, mass 1; collision box size=0.1 0.2 0.05; visual box size=0.1 0.05 0.1
- added link link1, mass 1; collision cylinder length=0.1 radius=0.05; visual cylinder length=0.1 radius=0.05
- added link link2, mass 1; collision cylinder length=0.3 radius=0.05; visual cylinder length=0.3 radius=0.05
- added link link3, mass 1; collision cylinder length=0.3 radius=0.05; visual cylinder length=0.3 radius=0.05
- added link link4, mass 1; collision cylinder length=0.3 radius=0.05; visual cylinder length=0.3 radius=0.05
- added link link5, mass 1; collision cylinder length=0.3 radius=0.05; visual cylinder length=0.3 radius=0.05
Joints:
- added joint hand_left_joint: type prismatic, parent gripper_base_link, child hand_left_link, origin xyz=0.0 -0.075 0.05 rpy=0 0 0, axis 0 1 0, limit lower=0 upper=0.05 effort=100 velocity=1, mimic joint=hand_right_joint
- added joint hand_right_joint: type prismatic, parent gripper_base_link, child hand_right_link, origin xyz=0.0 0.075 0.05 rpy=0 0 0, axis 0 -1 0, limit lower=0 upper=0.05 effort=100 velocity=1
- added joint joint1: type revolute, parent base_link, child link1, origin xyz=0.0 0.0 0.1 rpy=0 0 0, axis 0 0 1, limit lower=-3.14 upper=3.14 effort=100 velocity=1
- added joint joint2: type revolute, parent link1, child link2, origin xyz=0.0 0.0 0.1 rpy=0 0 0, axis 1 0 0, limit lower=-3.14 upper=3.14 effort=100 velocity=1
- added joint joint3: type revolute, parent link2, child link3, origin xyz=0.0 0.0 0.3 rpy=0 0 0, axis 1 0 0, limit lower=-3.14 upper=3.14 effort=100 velocity=1
- added joint joint4: type revolute, parent link3, child link4, origin xyz=0.0 0.0 0.3 rpy=0 0 0, axis 1 0 0, limit lower=-3.14 upper=3.14 effort=100 velocity=1
- added joint joint5: type revolute, parent link4, child link5, origin xyz=0.0 0.0 0.3 rpy=0 0 0, axis 1 0 0, limit lower=-3.14 upper=3.14 effort=100 velocity=1
- added joint joint6: type revolute, parent link5, child gripper_base_link, origin xyz=0.0 0.0 0.3 rpy=0 0 0, axis 0 0 1, limit lower=-3.14 upper=3.14 effort=100 velocity=1
